File: power.kicad_sch (KiCad schematic)
At the start: 84 parts, among them Q1 PJE138K, Q2 PJE138K, Q3 SSM3J332R, Q4 PJE138K, Q5 SSM3J332R, Q6 PJE138K, Q7 SSM3J332R, U1 TLV70018_SC70, U4 TPS65150PWP, U5 MPQ7235GQBE, U6 TLV76701_WSON6

Commit message: [#56078] Update symbols/footprints from lib
Parts:
- D11, D5, D8: value LED_G -> LED_G_0603_598-8D80-107F; footprint antmicro-footprints:LED_0603_1608Metric_R -> antmicro-footprints:LED_0603_1608Metric_G; symbol antmicroLEDIndicationDiscrete:LED_R_0603_598-8D80-107F -> antmicroLEDIndicationDiscrete:LED_G_0603_598-8D80-107F; Color (none) -> Green
- L1: DNP DNP -> (none)
- U6: value TLV76701_WSON6 -> TLV76701_WSON; symbol antmicroPMICVoltageRegulatorsLinear:TLV76701_WSON6 -> antmicroPMICVoltageRegulatorsLinear:TLV76701_WSON
Changed lines of the file:
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@@
     )
   )
-  (symbol (lib_id "antmicroLEDIndicationDiscrete:LED_R_0603_598-8D80-107F") (at 339.09 26.67 270) (unit 1)
+  (symbol (lib_id "antmicroLEDIndicationDiscrete:LED_G_0603_598-8D80-107F") (at 339.09 26.67 270) (unit 1)
     (in_bom yes) (on_board yes) (dnp no) (fields_autoplaced)
-    (property "Reference" "D11" (at 344.17 29.5274 90)
+    (property "Reference" "D11" (at 344.17 29.5275 90)
       (effects (font (size 1.27 1.27) (thickness 0.15)) (justify left))
     )
-    (property "Value" "LED_G" (at 344.17 32.0674 90)
-      (effects (font (size 1.27 1.27) (thickness 0.15)) (justify left))
+    (property "Value" "LED_G_0603_598-8D80-107F" (at 331.47 49.53 0)
+      (effects (font (size 1.27 1.27) (thickness 0.15)) (justify left bottom) hide)
     )
-    (property "Footprint" "antmicro-footprints:LED_0603_1608Metric_R" (at 331.47 49.53 0)
+    (property "Footprint" "antmicro-footprints:LED_0603_1608Metric_G" (at 328.93 49.53 0)
       (effects (font (size 1.27 1.27) (thickness 0.15)) (justify left bottom) hide)
     )
-    (property "Datasheet" "https://www.farnell.com/datasheets/3093797.pdf" (at 328.93 49.53 0)
+    (property "Datasheet" "https://www.farnell.com/datasheets/3093797.pdf" (at 326.39 49.53 0)
       (effects (font (size 1.27 1.27) (thickness 0.15)) (justify left bottom) hide)
     )
-    (property "MPN" "598-8D80-107F" (at 344.17 32.0674 90)
-      (effects (font (size 1.27 1.27) (thickness 0.15)) (justify left) hide)
+    (property "MPN" "598-8D80-107F" (at 323.85 49.53 0)
+      (effects (font (size 1.27 1.27) (thickness 0.15)) (justify left bottom) hide)
     )
-    (property "Manufacturer" "Dialight" (at 323.85 49.53 0)
+    (property "Manufacturer" "Dialight" (at 321.31 49.53 0)
       (effects (font (size 1.27 1.27) (thickness 0.15)) (justify left bottom) hide)
     )
-    (property "Author" "Antmicro" (at 321.31 49.53 0)
+    (property "Author" "Antmicro" (at 318.77 49.53 0)
       (effects (font (size 1.27 1.27) (thickness 0.15)) (justify left bottom) hide)
     )
-    (property "License" "Apache-2.0" (at 318.77 49.53 0)
+    (property "License" "Apache-2.0" (at 316.23 49.53 0)
       (effects (font (size 1.27 1.27) (thickness 0.15)) (justify left bottom) hide)
     )
+    (property "Color" "Green" (at 344.17 32.0675 90)
+      (effects (font (size 1.27 1.27)) (justify left))
+    )
     (pin "1")
     (pin "2")
@@
     )
   )
-  (symbol (lib_id "antmicroPMICVoltageRegulatorsLinear:TLV76701_WSON6") (at 293.37 128.27 0) (unit 1)
+  (symbol (lib_id "antmicroPMICVoltageRegulatorsLinear:TLV76701_WSON") (at 293.37 128.27 0) (unit 1)
     (in_bom yes) (on_board yes) (dnp no) (fields_autoplaced)
     (property "Reference" "U6" (at 300.99 120.65 0)
       (effects (font (size 1.27 1.27) (thickness 0.15)))
     )
-    (property "Value" "TLV76701_WSON6" (at 328.93 135.89 0)
+    (property "Value" "TLV76701_WSON" (at 328.93 135.89 0)
       (effects (font (size 1.27 1.27) (thickness 0.15)) (justify left bottom) hide)
     )
@@
     )
   )
-  (symbol (lib_id "antmicroLEDIndicationDiscrete:LED_R_0603_598-8D80-107F") (at 250.19 199.39 270) (unit 1)
+  (symbol (lib_id "antmicroLEDIndicationDiscrete:LED_G_0603_598-8D80-107F") (at 250.19 199.39 270) (unit 1)
     (in_bom yes) (on_board yes) (dnp no) (fields_autoplaced)
-    (property "Reference" "D8" (at 255.27 202.2474 90)
+    (property "Reference" "D8" (at 255.27 202.2475 90)
       (effects (font (size 1.27 1.27) (thickness 0.15)) (justify left))
     )
-    (property "Value" "LED_G" (at 255.27 204.7874 90)
-      (effects (font (size 1.27 1.27) (thickness 0.15)) (justify left))
+    (property "Value" "LED_G_0603_598-8D80-107F" (at 242.57 222.25 0)
+      (effects (font (size 1.27 1.27) (thickness 0.15)) (justify left bottom) hide)
     )
-    (property "Footprint" "antmicro-footprints:LED_0603_1608Metric_R" (at 242.57 222.25 0)
+    (property "Footprint" "antmicro-footprints:LED_0603_1608Metric_G" (at 240.03 222.25 0)
       (effects (font (size 1.27 1.27) (thickness 0.15)) (justify left bottom) hide)
     )
-    (property "Datasheet" "https://www.farnell.com/datasheets/3093797.pdf" (at 240.03 222.25 0)
+    (property "Datasheet" "https://www.farnell.com/datasheets/3093797.pdf" (at 237.49 222.25 0)
       (effects (font (size 1.27 1.27) (thickness 0.15)) (justify left bottom) hide)
     )
-    (property "MPN" "598-8D80-107F" (at 255.27 204.7874 90)
-      (effects (font (size 1.27 1.27) (thickness 0.15)) (justify left) hide)
+    (property "MPN" "598-8D80-107F" (at 234.95 222.25 0)
+      (effects (font (size 1.27 1.27) (thickness 0.15)) (justify left bottom) hide)
     )
-    (property "Manufacturer" "Dialight" (at 234.95 222.25 0)
+    (property "Manufacturer" "Dialight" (at 232.41 222.25 0)
       (effects (font (size 1.27 1.27) (thickness 0.15)) (justify left bottom) hide)
     )
-    (property "Author" "Antmicro" (at 232.41 222.25 0)
+    (property "Author" "Antmicro" (at 229.87 222.25 0)
       (effects (font (size 1.27 1.27) (thickness 0.15)) (justify left bottom) hide)
     )
-    (property "License" "Apache-2.0" (at 229.87 222.25 0)
+    (property "License" "Apache-2.0" (at 227.33 222.25 0)
       (effects (font (size 1.27 1.27) (thickness 0.15)) (justify left bottom) hide)
     )
+    (property "Color" "Green" (at 255.27 204.7875 90)
+      (effects (font (size 1.27 1.27)) (justify left))
+    )
     (pin "1")
     (pin "2")
@@
     )
   )
-  (symbol (lib_id "antmicroLEDIndicationDiscrete:LED_R_0603_598-8D80-107F") (at 124.46 205.74 270) (unit 1)
+  (symbol (lib_id "antmicroLEDIndicationDiscrete:LED_G_0603_598-8D80-107F") (at 124.46 205.74 270) (unit 1)
     (in_bom yes) (on_board yes) (dnp no) (fields_autoplaced)
     (property "Reference" "D5" (at 129.54 208.5975 90)
       (effects (font (size 1.27 1.27) (thickness 0.15)) (justify left))
     )
-    (property "Value" "LED_G" (at 129.54 211.1375 90)
-      (effects (font (size 1.27 1.27) (thickness 0.15)) (justify left))
+    (property "Value" "LED_G_0603_598-8D80-107F" (at 116.84 228.6 0)
+      (effects (font (size 1.27 1.27) (thickness 0.15)) (justify left bottom) hide)
     )
-    (property "Footprint" "antmicro-footprints:LED_0603_1608Metric_R" (at 116.84 228.6 0)
+    (property "Footprint" "antmicro-footprints:LED_0603_1608Metric_G" (at 114.3 228.6 0)
       (effects (font (size 1.27 1.27) (thickness 0.15)) (justify left bottom) hide)
     )
-    (property "Datasheet" "https://www.farnell.com/datasheets/3093797.pdf" (at 114.3 228.6 0)
+    (property "Datasheet" "https://www.farnell.com/datasheets/3093797.pdf" (at 111.76 228.6 0)
       (effects (font (size 1.27 1.27) (thickness 0.15)) (justify left bottom) hide)
     )
-    (property "MPN" "598-8D80-107F" (at 129.54 211.1374 90)
-      (effects (font (size 1.27 1.27) (thickness 0.15)) (justify left) hide)
+    (property "MPN" "598-8D80-107F" (at 109.22 228.6 0)
+      (effects (font (size 1.27 1.27) (thickness 0.15)) (justify left bottom) hide)
     )
-    (property "Manufacturer" "Dialight" (at 109.22 228.6 0)
+    (property "Manufacturer" "Dialight" (at 106.68 228.6 0)
       (effects (font (size 1.27 1.27) (thickness 0.15)) (justify left bottom) hide)
     )
-    (property "Author" "Antmicro" (at 106.68 228.6 0)
+    (property "Author" "Antmicro" (at 104.14 228.6 0)
       (effects (font (size 1.27 1.27) (thickness 0.15)) (justify left bottom) hide)
     )
-    (property "License" "Apache-2.0" (at 104.14 228.6 0)
+    (property "License" "Apache-2.0" (at 101.6 228.6 0)
       (effects (font (size 1.27 1.27) (thickness 0.15)) (justify left bottom) hide)
     )
+    (property "Color" "Green" (at 129.54 211.1375 90)
+      (effects (font (size 1.27 1.27)) (justify left))
+    )
     (pin "1")
     (pin "2")
@@
       (effects (font (size 1.27 1.27) (thickness 0.15)) (justify left bottom) hide)
     )
-    (property "DNP" "DNP" (at 190.5 53.34 0)
-      (effects (font (size 1.27 1.27)) hide)
-    )
     (pin "1")

Commit message: [#56708] Generate local library
Parts:
- C15: footprint antmicro-footprints:C_0402_1005Metric -> cm4-lvds-adapter-footprints:C_0402_1005Metric; symbol antmicroCapacitors0402:C_10u_0402 -> cm4-lvds-adapter:C_10u_0402
- C16, C2, C22, C3, C34, C35: footprint antmicro-footprints:C_0402_1005Metric -> cm4-lvds-adapter-footprints:C_0402_1005Metric; symbol antmicroCapacitors0402:C_1u_0402 -> cm4-lvds-adapter:C_1u_0402
- C17, C37: footprint antmicro-footprints:C_0402_1005Metric -> cm4-lvds-adapter-footprints:C_0402_1005Metric; symbol antmicroCapacitors0402:C_220n_16V_0402 -> cm4-lvds-adapter:C_220n_16V_0402
- C18, C19, C27, C31, C32, C36: footprint antmicro-footprints:C_0402_1005Metric -> cm4-lvds-adapter-footprints:C_0402_1005Metric; symbol antmicroCapacitors0402:C_100n_0402 -> cm4-lvds-adapter:C_100n_0402
- C20: footprint antmicro-footprints:C_0402_1005Metric -> cm4-lvds-adapter-footprints:C_0402_1005Metric; symbol antmicroCapacitors0402:C_2n2_0402 -> cm4-lvds-adapter:C_2n2_0402
- C21: footprint antmicro-footprints:C_0402_1005Metric -> cm4-lvds-adapter-footprints:C_0402_1005Metric; symbol antmicroCapacitors0402:C_1n_0402 -> cm4-lvds-adapter:C_1n_0402
- C23, C29, C30, C38, C41: footprint antmicro-footprints:C_0805_2012Metric -> cm4-lvds-adapter-footprints:C_0805_2012Metric; symbol antmicroCapacitorsmisc:C_22u_25V_0805 -> cm4-lvds-adapter:C_22u_25V_0805
- C24, C33: footprint antmicro-footprints:C_0402_1005Metric -> cm4-lvds-adapter-footprints:C_0402_1005Metric; symbol antmicroCapacitors0402:C_22p_0402 -> cm4-lvds-adapter:C_22p_0402
- C25: footprint antmicro-footprints:C_0402_1005Metric -> cm4-lvds-adapter-footprints:C_0402_1005Metric; symbol antmicroCapacitors0402:C_10n_0402 -> cm4-lvds-adapter:C_10n_0402
- C26, C28, C39, C40: footprint antmicro-footprints:C_0402_1005Metric -> cm4-lvds-adapter-footprints:C_0402_1005Metric; symbol antmicroCapacitors0402:C_1u_25V_0402 -> cm4-lvds-adapter:C_1u_25V_0402
- D10, D6: footprint antmicro-footprints:SOT-23-3 -> cm4-lvds-adapter-footprints:SOT-23-3; symbol antmicroDiodesRectifiersSingle:BAT54S-E3-08 -> cm4-lvds-adapter:BAT54S-E3-08
- D11, D5, D8: footprint antmicro-footprints:LED_0603_1608Metric_G -> cm4-lvds-adapter-footprints:LED_0603_1608Metric_G; symbol antmicroLEDIndicationDiscrete:LED_G_0603_598-8D80-107F -> cm4-lvds-adapter:LED_G_0603_598-8D80-107F
- D7: footprint antmicro-footprints:SOD-523 -> cm4-lvds-adapter-footprints:SOD-523; symbol antmicroDiodesRectifiersSingle:RB521S30T1G -> cm4-lvds-adapter:RB521S30T1G
- D9: footprint antmicro-footprints:D_SOD-323F -> cm4-lvds-adapter-footprints:D_SOD-323F; symbol antmicroDiodesRectifiersSingle:PMEG3010CE_SOD323 -> cm4-lvds-adapter:PMEG3010CE_SOD323
- L1: footprint antmicro-footprints:L_1008_2520Metric -> cm4-lvds-adapter-footprints:L_1008_2520Metric; symbol antmicroFixedInductors:L_3u3_2.5A_1008 -> cm4-lvds-adapter:L_3u3_2.5A_1008
- L2: footprint antmicro-footprints:L_Murata-8200 -> cm4-lvds-adapter-footprints:L_Murata-8200; symbol antmicroFixedInductors:L_10u_0.5A_Murata-8200 -> cm4-lvds-adapter:L_10u_0.5A_Murata-8200
- Q1, Q2, Q4, Q6: footprint antmicro-footprints:SOT-523 -> cm4-lvds-adapter-footprints:SOT-523; symbol antmicroTransistorsFETsMOSFETsSingle:PJE138K -> cm4-lvds-adapter:PJE138K
- Q3, Q5, Q7: footprint antmicro-footprints:SOT-23-3 -> cm4-lvds-adapter-footprints:SOT-23-3; symbol antmicroTransistorsFETsMOSFETsSingle:SSM3J332R -> cm4-lvds-adapter:SSM3J332R
- R10, R11, R17, R26, R33, R49: footprint antmicro-footprints:R_0402_1005Metric -> cm4-lvds-adapter-footprints:R_0402_1005Metric; symbol antmicroResistors0402:R_100k_0402 -> cm4-lvds-adapter:R_100k_0402
- R12, R20, R22, R23, R34, R35: footprint antmicro-footprints:R_0402_1005Metric -> cm4-lvds-adapter-footprints:R_0402_1005Metric; symbol antmicroResistors0402:R_0R_0402 -> cm4-lvds-adapter:R_0R_0402
- R13, R19: footprint antmicro-footprints:R_0402_1005Metric -> cm4-lvds-adapter-footprints:R_0402_1005Metric; symbol antmicroResistors0402:R_590k_0402 -> cm4-lvds-adapter:R_590k_0402
- R14: footprint antmicro-footprints:R_0402_1005Metric -> cm4-lvds-adapter-footprints:R_0402_1005Metric; symbol antmicroResistors0402:R_120k_0402 -> cm4-lvds-adapter:R_120k_0402
- R15, R30: footprint antmicro-footprints:R_0402_1005Metric -> cm4-lvds-adapter-footprints:R_0402_1005Metric; symbol antmicroResistors0402:R_330k_0402 -> cm4-lvds-adapter:R_330k_0402
- R16: footprint antmicro-footprints:R_0402_1005Metric -> cm4-lvds-adapter-footprints:R_0402_1005Metric; symbol antmicroResistors0402:R_49k9_0402 -> cm4-lvds-adapter:R_49k9_0402
- R18: footprint antmicro-footprints:R_0402_1005Metric -> cm4-lvds-adapter-footprints:R_0402_1005Metric; symbol antmicroResistors0402:R_1M_0402 -> cm4-lvds-adapter:R_1M_0402
- R21, R38: footprint antmicro-footprints:R_0402_1005Metric -> cm4-lvds-adapter-footprints:R_0402_1005Metric; symbol antmicroResistors0402:R_4k7_0402 -> cm4-lvds-adapter:R_4k7_0402
- R24, R37: footprint antmicro-footprints:R_0402_1005Metric -> cm4-lvds-adapter-footprints:R_0402_1005Metric; symbol antmicroResistors0402:R_10k_0402 -> cm4-lvds-adapter:R_10k_0402
- R25: footprint antmicro-footprints:R_0402_1005Metric -> cm4-lvds-adapter-footprints:R_0402_1005Metric; symbol antmicroResistors0402:R_820k_0402 -> cm4-lvds-adapter:R_820k_0402
- R27, R36: footprint antmicro-footprints:R_0402_1005Metric -> cm4-lvds-adapter-footprints:R_0402_1005Metric; symbol antmicroResistors0402:R_110k_0402 -> cm4-lvds-adapter:R_110k_0402
- R28: footprint antmicro-footprints:R_0402_1005Metric -> cm4-lvds-adapter-footprints:R_0402_1005Metric; symbol antmicroResistors0402:R_1M5_0402 -> cm4-lvds-adapter:R_1M5_0402
- R29: footprint antmicro-footprints:R_0603_1608Metric -> cm4-lvds-adapter-footprints:R_0603_1608Metric; symbol antmicroResistors0603:R_20R_0603 -> cm4-lvds-adapter:R_20R_0603
- R3, R9: footprint antmicro-footprints:R_0402_1005Metric -> cm4-lvds-adapter-footprints:R_0402_1005Metric; symbol antmicroResistors0402:R_1k_0402 -> cm4-lvds-adapter:R_1k_0402
- R31: footprint antmicro-footprints:R_0402_1005Metric -> cm4-lvds-adapter-footprints:R_0402_1005Metric; symbol antmicroResistors0402:R_1R2_0402 -> cm4-lvds-adapter:R_1R2_0402
- R32: footprint antmicro-footprints:R_0402_1005Metric -> cm4-lvds-adapter-footprints:R_0402_1005Metric; symbol antmicroResistors0402:R_510k_0402 -> cm4-lvds-adapter:R_510k_0402
- TP10: footprint antmicro-footprints:TP_SMD_0.75mm -> cm4-lvds-adapter-footprints:TP_SMD_0.75mm; symbol antmicroTestPoints:TP_0.75mm_SMD -> cm4-lvds-adapter:TP_0.75mm_SMD
- TP11, TP16: footprint antmicro-footprints:TP_SMD_1mm -> cm4-lvds-adapter-footprints:TP_SMD_1mm; symbol antmicroTestPoints:TP_1mm_SMD -> cm4-lvds-adapter:TP_1mm_SMD
- U1: footprint antmicro-footprints:SC-70-5 -> cm4-lvds-adapter-footprints:SC-70-5; symbol antmicroPMICVoltageRegulatorsLinear:TLV70018_SC70 -> cm4-lvds-adapter:TLV70018_SC70
- U4: footprint antmicro-footprints:HTSSOP-24_W4.4mm_P0.65mm -> cm4-lvds-adapter-footprints:HTSSOP-24_W4.4mm_P0.65mm; symbol antmicroPMICVoltageRegulatorsDCDCSwitchingRegulators:TPS65150_HTSSOP -> cm4-lvds-adapter:TPS65150_HTSSOP
- U5: footprint antmicro-footprints:QFN-13_2.5x3mm -> cm4-lvds-adapter-footprints:QFN-13_2.5x3mm; symbol antmicroPMICLEDDrivers:MPQ7235GQBE -> cm4-lvds-adapter:MPQ7235GQBE
- U6: footprint antmicro-footprints:WSON-6-1EP_2x2mm_P0.65mm -> cm4-lvds-adapter-footprints:WSON-6-1EP_2x2mm_P0.65mm; symbol antmicroPMICVoltageRegulatorsLinear:TLV76701_WSON -> cm4-lvds-adapter:TLV76701_WSON

Commit message: [#56708] Update symbol/footprint props; Fix J1 label
Parts:
- U4: value TPS65150PWP -> TPS65150_HTSSOP
Changed lines of the file:
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@@
     (effects (font (size 1.27 1.27)) (justify left bottom))
   )
-  (text "Delay here to let backlight \nshutdown before PMIC"
-    (at 88.9 57.15 0)
+  (text "Delay here to let backlight \nshutdown before PMIC" (at 88.9 57.15 0)
     (effects (font (size 1.27 1.27)) (justify left bottom))
   )
@@
       (effects (font (size 1.27 1.27) (thickness 0.15)))
     )
-    (property "Value" "TPS65150PWP" (at 220.98 57.15 0)
+    (property "Value" "TPS65150_HTSSOP" (at 220.98 57.15 0)
       (effects (font (size 1.27 1.27) (thickness 0.15)) (justify left bottom) hide)
     )

Commit message: [#57456] Remove loclib
Parts:
- C15: footprint cm4-lvds-adapter-footprints:C_0402_1005Metric -> antmicro-footprints:C_0402_1005Metric; symbol cm4-lvds-adapter:C_10u_0402 -> antmicroCapacitors0402:C_10u_0402
- C16, C2, C22, C3, C34, C35: footprint cm4-lvds-adapter-footprints:C_0402_1005Metric -> antmicro-footprints:C_0402_1005Metric; symbol cm4-lvds-adapter:C_1u_0402 -> antmicroCapacitors0402:C_1u_0402
- C17, C37: footprint cm4-lvds-adapter-footprints:C_0402_1005Metric -> antmicro-footprints:C_0402_1005Metric; symbol cm4-lvds-adapter:C_220n_16V_0402 -> antmicroCapacitors0402:C_220n_16V_0402
- C18, C19, C27, C31, C32, C36: footprint cm4-lvds-adapter-footprints:C_0402_1005Metric -> antmicro-footprints:C_0402_1005Metric; symbol cm4-lvds-adapter:C_100n_0402 -> antmicroCapacitors0402:C_100n_0402
- C20: footprint cm4-lvds-adapter-footprints:C_0402_1005Metric -> antmicro-footprints:C_0402_1005Metric; symbol cm4-lvds-adapter:C_2n2_0402 -> antmicroCapacitors0402:C_2n2_0402
- C21: footprint cm4-lvds-adapter-footprints:C_0402_1005Metric -> antmicro-footprints:C_0402_1005Metric; symbol cm4-lvds-adapter:C_1n_0402 -> antmicroCapacitors0402:C_1n_0402
- C23, C29, C30, C38, C41: footprint cm4-lvds-adapter-footprints:C_0805_2012Metric -> antmicro-footprints:C_0805_2012Metric; symbol cm4-lvds-adapter:C_22u_25V_0805 -> antmicroCapacitorsmisc:C_22u_25V_0805
- C24, C33: footprint cm4-lvds-adapter-footprints:C_0402_1005Metric -> antmicro-footprints:C_0402_1005Metric; symbol cm4-lvds-adapter:C_22p_0402 -> antmicroCapacitors0402:C_22p_0402
- C25: footprint cm4-lvds-adapter-footprints:C_0402_1005Metric -> antmicro-footprints:C_0402_1005Metric; symbol cm4-lvds-adapter:C_10n_0402 -> antmicroCapacitors0402:C_10n_0402
- C26, C28, C39, C40: footprint cm4-lvds-adapter-footprints:C_0402_1005Metric -> antmicro-footprints:C_0402_1005Metric; symbol cm4-lvds-adapter:C_1u_25V_0402 -> antmicroCapacitors0402:C_1u_25V_0402
- D10, D6: footprint cm4-lvds-adapter-footprints:SOT-23-3 -> antmicro-footprints:SOT-23-3; symbol cm4-lvds-adapter:BAT54S-E3-08 -> antmicroDiodesRectifiersSingle:BAT54S-E3-08
- D11, D5, D8: footprint cm4-lvds-adapter-footprints:LED_0603_1608Metric_G -> antmicro-footprints:LED_0603_1608Metric_G; symbol cm4-lvds-adapter:LED_G_0603_598-8D80-107F -> antmicroLEDIndicationDiscrete:LED_G_0603_598-8D80-107F
- D7: footprint cm4-lvds-adapter-footprints:SOD-523 -> antmicro-footprints:SOD-523; symbol cm4-lvds-adapter:RB521S30T1G -> antmicroDiodesRectifiersSingle:RB521S30T1G
- D9: footprint cm4-lvds-adapter-footprints:D_SOD-323F -> antmicro-footprints:D_SOD-323F; symbol cm4-lvds-adapter:PMEG3010CE_SOD323 -> antmicroDiodesRectifiersSingle:PMEG3010CE_SOD323
- L1: footprint cm4-lvds-adapter-footprints:L_1008_2520Metric -> antmicro-footprints:L_1008_2520Metric; symbol cm4-lvds-adapter:L_3u3_2.5A_1008 -> antmicroFixedInductors:L_3u3_2.5A_1008
- L2: footprint cm4-lvds-adapter-footprints:L_Murata-8200 -> antmicro-footprints:L_Murata-8200; symbol cm4-lvds-adapter:L_10u_0.5A_Murata-8200 -> antmicroFixedInductors:L_10u_0.5A_Murata-8200
- Q1, Q2, Q4, Q6: footprint cm4-lvds-adapter-footprints:SOT-523 -> antmicro-footprints:SOT-523; symbol cm4-lvds-adapter:PJE138K -> antmicroTransistorsFETsMOSFETsSingle:PJE138K
- Q3, Q5, Q7: footprint cm4-lvds-adapter-footprints:SOT-23-3 -> antmicro-footprints:SOT-23-3; symbol cm4-lvds-adapter:SSM3J332R -> antmicroTransistorsFETsMOSFETsSingle:SSM3J332R
- R10, R11, R17, R26, R33, R49: footprint cm4-lvds-adapter-footprints:R_0402_1005Metric -> antmicro-footprints:R_0402_1005Metric; symbol cm4-lvds-adapter:R_100k_0402 -> antmicroResistors0402:R_100k_0402
- R12, R20, R22, R23, R34, R35: footprint cm4-lvds-adapter-footprints:R_0402_1005Metric -> antmicro-footprints:R_0402_1005Metric; symbol cm4-lvds-adapter:R_0R_0402 -> antmicroResistors0402:R_0R_0402
- R13, R19: footprint cm4-lvds-adapter-footprints:R_0402_1005Metric -> antmicro-footprints:R_0402_1005Metric; symbol cm4-lvds-adapter:R_590k_0402 -> antmicroResistors0402:R_590k_0402
- R14: footprint cm4-lvds-adapter-footprints:R_0402_1005Metric -> antmicro-footprints:R_0402_1005Metric; symbol cm4-lvds-adapter:R_120k_0402 -> antmicroResistors0402:R_120k_0402
- R15, R30: footprint cm4-lvds-adapter-footprints:R_0402_1005Metric -> antmicro-footprints:R_0402_1005Metric; symbol cm4-lvds-adapter:R_330k_0402 -> antmicroResistors0402:R_330k_0402
- R16: footprint cm4-lvds-adapter-footprints:R_0402_1005Metric -> antmicro-footprints:R_0402_1005Metric; symbol cm4-lvds-adapter:R_49k9_0402 -> antmicroResistors0402:R_49k9_0402
- R18: footprint cm4-lvds-adapter-footprints:R_0402_1005Metric -> antmicro-footprints:R_0402_1005Metric; symbol cm4-lvds-adapter:R_1M_0402 -> antmicroResistors0402:R_1M_0402
- R21, R38: footprint cm4-lvds-adapter-footprints:R_0402_1005Metric -> antmicro-footprints:R_0402_1005Metric; symbol cm4-lvds-adapter:R_4k7_0402 -> antmicroResistors0402:R_4k7_0402
- R24, R37: footprint cm4-lvds-adapter-footprints:R_0402_1005Metric -> antmicro-footprints:R_0402_1005Metric; symbol cm4-lvds-adapter:R_10k_0402 -> antmicroResistors0402:R_10k_0402
- R25: footprint cm4-lvds-adapter-footprints:R_0402_1005Metric -> antmicro-footprints:R_0402_1005Metric; symbol cm4-lvds-adapter:R_820k_0402 -> antmicroResistors0402:R_820k_0402
- R27, R36: footprint cm4-lvds-adapter-footprints:R_0402_1005Metric -> antmicro-footprints:R_0402_1005Metric; symbol cm4-lvds-adapter:R_110k_0402 -> antmicroResistors0402:R_110k_0402
- R28: footprint cm4-lvds-adapter-footprints:R_0402_1005Metric -> antmicro-footprints:R_0402_1005Metric; symbol cm4-lvds-adapter:R_1M5_0402 -> antmicroResistors0402:R_1M5_0402
- R29: footprint cm4-lvds-adapter-footprints:R_0603_1608Metric -> antmicro-footprints:R_0603_1608Metric; symbol cm4-lvds-adapter:R_20R_0603 -> antmicroResistors0603:R_20R_0603
- R3, R9: footprint cm4-lvds-adapter-footprints:R_0402_1005Metric -> antmicro-footprints:R_0402_1005Metric; symbol cm4-lvds-adapter:R_1k_0402 -> antmicroResistors0402:R_1k_0402
- R31: footprint cm4-lvds-adapter-footprints:R_0402_1005Metric -> antmicro-footprints:R_0402_1005Metric; symbol cm4-lvds-adapter:R_1R2_0402 -> antmicroResistors0402:R_1R2_0402
- R32: footprint cm4-lvds-adapter-footprints:R_0402_1005Metric -> antmicro-footprints:R_0402_1005Metric; symbol cm4-lvds-adapter:R_510k_0402 -> antmicroResistors0402:R_510k_0402
- TP10: footprint cm4-lvds-adapter-footprints:TP_SMD_0.75mm -> antmicro-footprints:TP_SMD_0.75mm; symbol cm4-lvds-adapter:TP_0.75mm_SMD -> antmicroTestPoints:TP_0.75mm_SMD
- TP11, TP16: footprint cm4-lvds-adapter-footprints:TP_SMD_1mm -> antmicro-footprints:TP_SMD_1mm; symbol cm4-lvds-adapter:TP_1mm_SMD -> antmicroTestPoints:TP_1mm_SMD
- U1: footprint cm4-lvds-adapter-footprints:SC-70-5 -> antmicro-footprints:SC-70-5; symbol cm4-lvds-adapter:TLV70018_SC70 -> antmicroPMICVoltageRegulatorsLinear:TLV70018_SC70
- U4: footprint cm4-lvds-adapter-footprints:HTSSOP-24_W4.4mm_P0.65mm -> antmicro-footprints:HTSSOP-24_W4.4mm_P0.65mm; symbol cm4-lvds-adapter:TPS65150_HTSSOP -> antmicroPMICVoltageRegulatorsDCDCSwitchingRegulators:TPS65150_HTSSOP
- U5: footprint cm4-lvds-adapter-footprints:QFN-13_2.5x3mm -> antmicro-footprints:QFN-13_2.5x3mm; symbol cm4-lvds-adapter:MPQ7235GQBE -> antmicroPMICLEDDrivers:MPQ7235GQBE
- U6: footprint cm4-lvds-adapter-footprints:WSON-6-1EP_2x2mm_P0.65mm -> antmicro-footprints:WSON-6-1EP_2x2mm_P0.65mm; symbol cm4-lvds-adapter:TLV76701_WSON -> antmicroPMICVoltageRegulatorsLinear:TLV76701_WSON
