File: cm4-lvds-adapter.kicad_pcb (KiCad board)
At the start: 6 copper layers, 52 x 43 mm, 155 parts, among them J1 Plug_Molex_SlimStack_2x20_556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, J2 JST_SUR_1x10_SM10B-SURS-TF-LF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, J3 FFC_Amphenol_1x40_62684-40110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, Q1 PJE138K, Q2 PJE138K, Q3 SSM3J332R, Q4 PJE138K, Q5 SSM3J332R, Q6 PJE138K, Q7 SSM3J332R, Q8 PJE138K, U1 TLV70018_SC70, U2 NTS0104_DHVQFN, U3 SN65DSI84, U4 TPS65150_HTSSOP, U5 MPQ7235GQBE, U6 TLV76701_WSON

Commit message: [#73840] Update 3V3 LED resistors to 100R andd 10V5 LED resistors to 1k5
Parts:
- R2, R21: value R_1k_0402 -> R_1k5_0402
- R3: value R_330R_0402 -> R_100R_0402
